Commit message: Sync workspace packages and stabilize autonomous navigation

File: diadem_description/urdf/diadem.xacro (robot description, xacro)
@@ -7,6 +7,6 @@
   <inertial>
     <origin xyz="-0.000442563326493991 0.0005036289593653383 0.2715469717743787" rpy="0 0 0"/>
-    <mass value="46.062115064028625"/>
-    <inertia ixx="2.183508" iyy="3.678419" izz="5.108526" ixy="0.008815" iyz="-0.001381" ixz="-0.002933"/>
+    <mass value="120.00"/>
+    <inertia ixx="5.68" iyy="9.60" izz="13.28" ixy="0.0228" iyz="-0.0036" ixz="-0.0076"/>
   </inertial>
   <visual>
@@ -17,8 +17,8 @@
     <material name="silver"/>
   </visual>
-  <collision>
-    <origin xyz="0 0 0" rpy="0 0 0"/>
+  <collision name="base_link_collision">
+    <origin xyz="0 0 0.25" rpy="0 0 0"/>
     <geometry>
-      <mesh filename="package://diadem_description/meshes/base_link.dae" scale="0.001 0.001 0.001"/>
+      <box size="0.5 0.5 0.3"/>
     </geometry>
   </collision>
@@ -37,8 +37,8 @@
     <material name="silver"/>
   </visual>
-  <collision>
-    <origin xyz="0.28 0.3 -0.18" rpy="0 0 0"/>
+  <collision name="RR_wheel_1_collision">
+    <origin xyz="0 0 0" rpy="1.57079632679 0 0"/>
     <geometry>
-      <mesh filename="package://diadem_description/meshes/RR_wheel_1.dae" scale="0.001 0.001 0.001"/>
+      <cylinder radius="0.18" length="0.08"/>
     </geometry>
   </collision>
@@ -57,8 +57,29 @@
     <material name="silver"/>
   </visual>
+  <collision name="FL_wheel_1_collision">
+    <origin xyz="0 0 0" rpy="1.57079632679 0 0"/>
+    <geometry>
+      <cylinder radius="0.18" length="0.08"/>
+    </geometry>
+  </collision>
+</link>
+<!-- Add this LiDAR link after the existing links -->
+<link name="lidar">
+  <inertial>
+    <origin xyz="0 0 0" rpy="0 0 0"/>
+    <mass value="0.5"/>
+    <inertia ixx="0.001" iyy="0.001" izz="0.001" ixy="0.0" iyz="0.0" ixz="0.0"/>
+  </inertial>
+  <visual>
+    <origin xyz="0 0 0" rpy="0 0 0"/>
+    <geometry>
+      <cylinder radius="0.05" length="0.06"/>
+    </geometry>
+    <material name="black"/>
+  </visual>
   <collision>
-    <origin xyz="-0.28 -0.3 -0.18" rpy="0 0 0"/>
+    <origin xyz="0 0 0" rpy="0 0 0"/>
     <geometry>
-      <mesh filename="package://diadem_description/meshes/FL_wheel_1.dae" scale="0.001 0.001 0.001"/>
+      <cylinder radius="0.05" length="0.06"/>
     </geometry>
   </collision>
@@ -77,8 +98,8 @@
     <material name="silver"/>
   </visual>
-  <collision>
-    <origin xyz="0.28 -0.3 -0.18" rpy="0 0 0"/>
+  <collision name="RL_wheel_1_collision">
+    <origin xyz="0 0 0" rpy="1.57079632679 0 0"/>
     <geometry>
-      <mesh filename="package://diadem_description/meshes/RL_wheel_1.dae" scale="0.001 0.001 0.001"/>
+      <cylinder radius="0.18" length="0.08"/>
     </geometry>
   </collision>
@@ -97,12 +118,13 @@
     <material name="silver"/>
   </visual>
-  <collision>
-    <origin xyz="-0.28 0.3 -0.18" rpy="0 0 0"/>
+  <collision name="FR_wheel_1_collision">
+    <origin xyz="0 0 0" rpy="1.57079632679 0 0"/>
     <geometry>
-      <mesh filename="package://diadem_description/meshes/FR_wheel_1.dae" scale="0.001 0.001 0.001"/>
+      <cylinder radius="0.18" length="0.08"/>
     </geometry>
   </collision>
 </link>
 <link name="imu_link"/>
+<link name="camera_link"/>
 <joint name="imu_joint" type="fixed">
     <origin rpy="0 0 0" xyz="0.0 0.0 0.310"/>
@@ -128,4 +150,10 @@
   <axis xyz="-0.0 1.0 0.0"/>
 </joint>
+<!-- Add this LiDAR joint after the existing joints -->
+<joint name="lidar_joint" type="fixed">
+  <origin xyz="0.0 0.0 0.64" rpy="0 0 0"/>
+  <parent link="base_link"/>
+  <child link="lidar"/>
+</joint>
 <joint name="FR_wheel_joint" type="continuous">
   <origin xyz="0.28 -0.3 0.18" rpy="0 0 0"/>
@@ -134,3 +162,8 @@
   <axis xyz="-0.0 1.0 -0.0"/>
 </joint>
+  <joint name="camera_joint" type="fixed">
+    <parent link="base_link"/>
+    <child link="camera_link"/>
+    <origin xyz="0 0 0.94" rpy="0.0 0.45 0"/>
+  </joint>
 </robot>

File: diadem_description/urdf/diadem_sim.xacro (robot description, xacro)
@@ -7,6 +7,6 @@
   <inertial>
     <origin xyz="-0.000442563326493991 0.0005036289593653383 0.2715469717743787" rpy="0 0 0"/>
-    <mass value="46.062115064028625"/>
-    <inertia ixx="2.183508" iyy="3.678419" izz="5.108526" ixy="0.008815" iyz="-0.001381" ixz="-0.002933"/>
+    <mass value="120.00"/>
+    <inertia ixx="5.68" iyy="9.60" izz="13.28" ixy="0.0228" iyz="-0.0036" ixz="-0.0076"/>
   </inertial>
   <visual>
@@ -17,8 +17,8 @@
     <material name="silver"/>
   </visual>
-  <collision>
-    <origin xyz="0 0 0" rpy="0 0 0"/>
+  <collision name="base_link_collision">
+    <origin xyz="0 0 0.25" rpy="0 0 0"/>
     <geometry>
-      <mesh filename="file://$(find diadem_description)/meshes/base_link.dae" scale="0.001 0.001 0.001"/>
+      <box size="0.5 0.5 0.3"/>
     </geometry>
   </collision>
@@ -37,8 +37,8 @@
     <material name="silver"/>
   </visual>
-  <collision>
-    <origin xyz="0.28 0.3 -0.18" rpy="0 0 0"/>
+  <collision name="RR_wheel_1_collision">
+    <origin xyz="0 0 0" rpy="1.57079632679 0 0"/>
     <geometry>
-      <mesh filename="file://$(find diadem_description)/meshes/RR_wheel_1.dae" scale="0.001 0.001 0.001"/>
+      <cylinder radius="0.18" length="0.08"/>
     </geometry>
   </collision>
@@ -57,8 +57,8 @@
     <material name="silver"/>
   </visual>
-  <collision>
-    <origin xyz="-0.28 -0.3 -0.18" rpy="0 0 0"/>
+  <collision name="FL_wheel_1_collision">
+    <origin xyz="0 0 0" rpy="1.57079632679 0 0"/>
     <geometry>
-      <mesh filename="file://$(find diadem_description)/meshes/FL_wheel_1.dae" scale="0.001 0.001 0.001"/>
+      <cylinder radius="0.18" length="0.08"/>
     </geometry>
   </collision>
@@ -77,8 +77,29 @@
     <material name="silver"/>
   </visual>
+  <collision name="RL_wheel_1_collision">
+    <origin xyz="0 0 0" rpy="1.57079632679 0 0"/>
+    <geometry>
+      <cylinder radius="0.18" length="0.08"/>
+    </geometry>
+  </collision>
+</link>
+<!-- Add this LiDAR link after the existing links -->
+<link name="lidar">
+  <inertial>
+    <origin xyz="0 0 0" rpy="0 0 0"/>
+    <mass value="0.5"/>
+    <inertia ixx="0.001" iyy="0.001" izz="0.001" ixy="0.0" iyz="0.0" ixz="0.0"/>
+  </inertial>
+  <visual>
+    <origin xyz="0 0 0" rpy="0 0 0"/>
+    <geometry>
+      <cylinder radius="0.05" length="0.06"/>
+    </geometry>
+    <material name="black"/>
+  </visual>
   <collision>
-    <origin xyz="0.28 -0.3 -0.18" rpy="0 0 0"/>
+    <origin xyz="0 0 0" rpy="0 0 0"/>
     <geometry>
-      <mesh filename="file://$(find diadem_description)/meshes/RL_wheel_1.dae" scale="0.001 0.001 0.001"/>
+      <cylinder radius="0.05" length="0.06"/>
     </geometry>
   </collision>
@@ -97,8 +118,8 @@
     <material name="silver"/>
   </visual>
-  <collision>
-    <origin xyz="-0.28 0.3 -0.18" rpy="0 0 0"/>
+  <collision name="FR_wheel_1_collision">
+    <origin xyz="0 0 0" rpy="1.57079632679 0 0"/>
     <geometry>
-      <mesh filename="file://$(find diadem_description)/meshes/FR_wheel_1.dae" scale="0.001 0.001 0.001"/>
+      <cylinder radius="0.18" length="0.08"/>
     </geometry>
   </collision>
@@ -134,3 +155,8 @@
   <axis xyz="-0.0 1.0 -0.0"/>
 </joint>
+<joint name="lidar_joint" type="fixed">
+  <origin xyz="0.0 0.0 0.64" rpy="0 0 -0.06"/>
+  <parent link="base_link"/>
+  <child link="lidar"/>
+</joint>
 </robot>

File: diadem_description/urdf/materials.xacro (robot description, xacro)
@@ -4,3 +4,6 @@
   <color rgba="0.700 0.700 0.700 1.000"/>
 </material>
+<material name="black">
+  <color rgba="0 0 0 1"/>
+</material>
 </robot>
